File: eagle/smd/kelvin_ntc_B.sch (EAGLE design)
At the start: 49 parts, among them IC1 PIC18F2580, IC3 MCP2551SN, IC4 LM2575S, J1 OSTTE-12, J2 A00-108-220-450, Q1 10 MHz

Commit message: Added missing files
Connections:
- net N$22 renamed CANH
Changed lines of the file:
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@@
 <?xml version="1.0" encoding="utf-8"?>
 <!DOCTYPE eagle SYSTEM "eagle.dtd">
-<eagle version="6.5.0">
+<eagle version="6.6.0">
 <drawing>
 <settings>
@@
 </segment>
 </net>
-<net name="N$22" class="0">
+<net name="CANH" class="0">
 <segment>
 <wire x1="269.24" y1="243.84" x2="269.24" y2="238.76" width="0.1524" layer="91"/>

Commit message: C14 should be 10K
Parts:
- C14: value 1 uF -> 10 uF
Changed lines of the file:
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@@
 <part name="C13" library="rcl" deviceset="C-EU" device="C0805" value="10uF"/>
 <part name="GND31" library="SUPPLY1" deviceset="GND" device=""/>
-<part name="C14" library="rcl" deviceset="C-EU" device="C0805" value="1 uF"/>
+<part name="C14" library="rcl" deviceset="C-EU" device="C0805" value="10 uF"/>
 <part name="GND32" library="SUPPLY1" deviceset="GND" device=""/>
 <part name="R17" library="rcl" deviceset="R-EU_" device="R0805" value="120"/>
